File: hardware/KiCAD-Keyboard-Tutorial-master/tutorial.kicad_pcb (KiCad board)
At the start: 2 copper layers, 284.5 x 94 mm, 65 parts, among them SW0:0 CTRL, SW0:1 SUPER, SW0:2 ALT, SW0:4 SPACE, SW1:1 SHIFT, SW1:2 Z, SW1:3 X, SW1:4 C, SW1:5 V, SW1:6 B, SW2:0 CAPS, SW2:1 A, SW2:2 S, SW2:3 D, SW2:4 F, SW2:5 G, SW2:6 H, SW3:0 TAB, SW3:1 Q, SW3:2 W, SW3:3 E, SW3:4 R, SW3:5 T, SW3:6 Y, SW4:0 TILDE, SW4:1 1, SW4:2 2, SW4:3 3, SW4:4 4, SW4:5 5, SW4:6 6, U1 TEENSY2.0

Commit message: pcb designed 1
Parts:
- removed D1:5, D1:6, D2:5, D2:6, D3:5, D3:6, D4:5, D4:6: D, footprints:DIODE
- removed Display1: sh1106, Connector_PinSocket_2.54mm:PinSocket_1x04_P2.54mm_Vertical
- removed SW1:5: V, footprints:CHERRY_PCB_100H
- removed SW1:6: B, footprints:CHERRY_PCB_100H
- removed SW2:5: G, footprints:CHERRY_PCB_100H
- removed SW2:6: H, footprints:CHERRY_PCB_100H
- removed SW3:5: T, footprints:CHERRY_PCB_100H
- removed SW3:6: Y, footprints:CHERRY_PCB_100H
- removed SW4:5: 5, footprints:CHERRY_PCB_100H
- removed SW4:6: 6, footprints:CHERRY_PCB_100H
- removed U1: TEENSY2.0, footprints:TEENSY_2.0
- added DISPLAY1: sh1106, user_footprints:4pin oled display 1,3, F.Cu at (491.1, 44.8)
- added EN1: Rotary_Encoder_Switch, Rotary_Encoder:RotaryEncoder_Alps_EC12E-Switch_Vertical_H20mm, F.Cu at (483.6, 113.7)
- added EN2: Rotary_Encoder_Switch, Rotary_Encoder:RotaryEncoder_Alps_EC12E-Switch_Vertical_H20mm, F.Cu at (347.4, 90.1)
- added MCU1: Pico, MCU_RaspberryPi_and_Boards:RPi_Pico_SMD_TH, F.Cu at (351.0, 48.6)
- SW0:0, SW0:1, SW0:2: footprint footprints:CHERRY_PCB_125H -> footprints:CHERRY_PCB_100H
- SW0:4: footprint footprints:CHERRY_PCB_275H -> footprints:CHERRY_PCB_200H
- SW1:1: footprint footprints:CHERRY_PCB_225H -> footprints:CHERRY_PCB_200H
- SW2:0: footprint footprints:CHERRY_PCB_175H -> footprints:CHERRY_PCB_100H
- SW3:0: footprint footprints:CHERRY_PCB_150H -> footprints:CHERRY_PCB_100H
- moved SW:WHEEL1 468.9 mm to (491.1, 78.1)
- moved SW4:1 329.4 mm to (399.1, 40.0)
- moved SW4:2 329.4 mm to (418.1, 40.0)
- moved SW4:0 329.4 mm to (380.0, 40.0)
- moved SW4:3 329.4 mm to (437.1, 40.0)
- moved SW4:4 329.4 mm to (456.2, 40.0)
- moved D4:1 328.4 mm to (389.8, 40.0), turned to 90 degrees
- moved D4:2 328.4 mm to (408.8, 40.0), turned to 90 degrees
- moved D4:3 328.4 mm to (427.9, 40.0), turned to 90 degrees
- moved D4:4 328.4 mm to (446.9, 40.0), turned to 90 degrees
- moved SW0:0 327.0 mm to (380.0, 116.2)
- moved SW1:1 327.0 mm to (389.5, 97.2)
- moved SW1:2 324.6 mm to (418.1, 97.2)
- moved SW1:3 324.6 mm to (437.1, 97.2)
- moved SW1:4 324.6 mm to (456.2, 97.2)
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Connections:
- SW:WHEEL1 pad 1: Net-(SW:WHEEL1-Pad1) -> GND
- SW:WHEEL1 pad 2: Net-(SW:WHEEL1-Pad2) -> /SW_WHEEL
Routing:
- net /ROW2: track 139.2 -> 0.00 mm
- net /ROW3: track 136.8 -> 0.00 mm
- net /ROW4: track 132.1 -> 0.00 mm
- net /ROW1: track 121.4 -> 0.00 mm
- net /COL1: track 103.0 -> 0.00 mm
- net /COL4: track 99.6 -> 0.00 mm
- net /COL2: track 98.6 -> 0.00 mm
- net /ROW0: track 98.4 -> 0.00 mm
- net /COL0: track 90.4 -> 0.00 mm
- net /COL5: track 73.5 -> 0.00 mm
- net /COL6: track 73.5 -> 0.00 mm
- net /COL3: track 73.5 -> 0.00 mm
- net Net-(D0:4-Pad1): track 26.0 -> 0.00 mm
- net Net-(D1:1-Pad1): track 23.2 -> 0.00 mm
- net Net-(D3:0-Pad1): track 13.7 -> 0.00 mm
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Other:
- board size 284.5 x 94 mm -> 185.7 x 106 mm

Commit message: pcb polished
Parts:
- added hole1: MountingHole_3.2mm_M3, MountingHole:MountingHole_3.2mm_M3, F.Cu at (330.4, 28.5)
- added hole1: MountingHole_3.2mm_M3, MountingHole:MountingHole_3.2mm_M3, F.Cu at (512.0, 127.0)
- added hole1: MountingHole_3.2mm_M3, MountingHole:MountingHole_3.2mm_M3, F.Cu at (330.4, 127.0)
- added hole1: MountingHole_3.2mm_M3, MountingHole:MountingHole_3.2mm_M3, F.Cu at (472.0, 78.1)
- moved EN1 11.2 mm to (488.6, 123.7), turned to 90 degrees
- turned SW:WHEEL1 to 225 degrees
Connections:
- MCU1 pad 1: Net-(MCU1-Pad1) -> /SW_WHEEL
- MCU1 pad 15: /COL0 -> Net-(MCU1-Pad15)
- MCU1 pad 16: /COL1 -> Net-(MCU1-Pad16)
- MCU1 pad 17: /COL2 -> Net-(MCU1-Pad17)
- MCU1 pad 19: /COL3 -> Net-(MCU1-Pad19)
- MCU1 pad 2: Net-(MCU1-Pad2) -> /EN1_SW
- MCU1 pad 20: /COL4 -> /EN2_SW
- MCU1 pad 21: /ROW4 -> /ROW0
- MCU1 pad 22: /ROW3 -> /ROW1
- MCU1 pad 25: /ROW1 -> /ROW3
- MCU1 pad 26: /ROW0 -> /ROW4
- MCU1 pad 27: /SW_WHEEL -> /COL0
- MCU1 pad 29: Net-(MCU1-Pad29) -> /COL1
- MCU1 pad 31: /EN1_SW -> /COL2
- MCU1 pad 32: /EN2_SW -> /COL3
- MCU1 pad 34: Net-(MCU1-Pad34) -> /COL4
- MCU1 pad 4: /EN1_B -> /EN2_B
- MCU1 pad 5: /EN1_A -> /EN2_A
- MCU1 pad 6: /EN2_B -> /EN1_B
- MCU1 pad 7: /EN2_A -> /EN1_A
Routing:
- net /SW_WHEEL: track 0.00 -> 311.4 mm
- net /SDA: track 0.00 -> 288.5 mm
- net /EN1_SW: track 0.00 -> 279.9 mm
- net GND: track 0.00 -> 275.1 mm
- net /SCL: track 0.00 -> 273.2 mm
- net /EN1_B: track 0.00 -> 230.9 mm
- net /EN1_A: track 0.00 -> 229.1 mm
- net /COL4: track 0.00 -> 187.7 mm
- net /COL2: track 0.00 -> 141.7 mm
- net /COL1: track 0.00 -> 141.7 mm
- net /COL3: track 0.00 -> 139.6 mm
- net VCC: track 0.00 -> 133.2 mm
- net /ROW0: track 0.00 -> 124.0 mm
- net /ROW4: track 0.00 -> 117.3 mm
- net /ROW1: track 0.00 -> 111.6 mm
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Other:
- board size 185.7 x 106 mm -> 191.6 x 108.5 mm
