File: hardware/KiCAD-Keyboard-Tutorial-master/tutorial.sch (KiCad schematic (older format))
At the start: 65 parts, among them SW0:0 CTRL, SW0:1 SUPER, SW0:2 ALT, SW0:4 SPACE, SW1:1 SHIFT, SW1:2 Z, SW1:3 X, SW1:4 C, SW1:5 V, SW1:6 B, SW2:0 CAPS, SW2:1 A, SW2:2 S, SW2:3 D, SW2:4 F, SW2:5 G, SW2:6 H, SW3:0 TAB, SW3:1 Q, SW3:2 W, SW3:3 E, SW3:4 R, SW3:5 T, SW3:6 Y, SW4:0 TILDE, SW4:1 1, SW4:2 2, SW4:3 3, SW4:4 4, SW4:5 5, SW4:6 6, U1 TEENSY2.0

Commit message: pcb designed 1
Parts:
- removed D1:5, D1:6, D2:5, D2:6, D3:5, D3:6, D4:5, D4:6: D, footprints:DIODE, symbol tutorial-rescue:DIODE
- removed Display1: sh1106, Connector_PinSocket_2.54mm:PinSocket_1x04_P2.54mm_Vertical, symbol userLibrary:sh1106
- removed SW1:5: V, footprints:CHERRY_PCB_100H, symbol tutorial-rescue:SWITCH_PUSH
- removed SW1:6: B, footprints:CHERRY_PCB_100H, symbol tutorial-rescue:SWITCH_PUSH
- removed SW2:5: G, footprints:CHERRY_PCB_100H, symbol tutorial-rescue:SWITCH_PUSH
- removed SW2:6: H, footprints:CHERRY_PCB_100H, symbol tutorial-rescue:SWITCH_PUSH
- removed SW3:5: T, footprints:CHERRY_PCB_100H, symbol tutorial-rescue:SWITCH_PUSH
- removed SW3:6: Y, footprints:CHERRY_PCB_100H, symbol tutorial-rescue:SWITCH_PUSH
- removed SW4:5: 5, footprints:CHERRY_PCB_100H, symbol tutorial-rescue:SWITCH_PUSH
- removed SW4:6: 6, footprints:CHERRY_PCB_100H, symbol tutorial-rescue:SWITCH_PUSH
- removed U1: TEENSY2.0, footprints:TEENSY_2.0, symbol tutorial-rescue:TEENSY2.0
- added DISPLAY: sh1106, user_footprints:4pin oled display 1,3, symbol userLibrary:sh1106
- added EN1, EN2: Rotary_Encoder_Switch, Rotary_Encoder:RotaryEncoder_Alps_EC12E-Switch_Vertical_H20mm, symbol Device:Rotary_Encoder_Switch
- added MCU: Pico, MCU_RaspberryPi_and_Boards:RPi_Pico_SMD_TH, symbol MCU_RaspberryPi_and_Boards:Pico
Connections:
- net COL0: now also MCU.15 (GPIO11)
- net COL1: now also MCU.16 (GPIO12)
- net COL2: now also MCU.17 (GPIO13)
- net COL3: now also MCU.19 (GPIO14)
- net COL4: now also MCU.20 (GPIO15)
- net GND: now also SW:WHEEL1.1, DISPLAY.2 (GND), EN1.C, EN1.S2, EN2.C, EN2.S2, MCU.13 (GND), MCU.18 (GND), MCU.23 (GND), MCU.28 (GND), MCU.3 (GND), MCU.33 (AGND), MCU.38 (GND), MCU.8 (GND)
- net ROW0: now also MCU.26 (GPIO20)
- net ROW1: now also MCU.25 (GPIO19)
- net ROW2: now also MCU.24 (GPIO18)
- net ROW3: now also MCU.22 (GPIO17)
- net ROW4: now also MCU.21 (GPIO16)
- net VCC: now also DISPLAY.1 (vcc), MCU.36 (3V3)
- net SW_WHEEL: now reaches SW:WHEEL1.2
- net SW_WHEEL: now also MCU.27 (GPIO21)
- new net EN1_A: EN1.A, MCU.5 (GPIO3)
- new net EN1_B: EN1.B, MCU.4 (GPIO2)
- new net EN1_SW: EN1.S1, MCU.31 (GPIO26_ADC0)
- new net EN2_A: EN2.A, MCU.7 (GPIO5)
- new net EN2_B: EN2.B, MCU.6 (GPIO4)
- new net EN2_SW: EN2.S1, MCU.32 (GPIO27_ADC1)
- new net SCL: DISPLAY.3 (SCL), MCU.12 (GPIO9)
- new net SDA: DISPLAY.4 (SDA), MCU.11 (GPIO8)
- no-connect marks 2 -> 0
Other:
- moved on the sheet: D0:0, D0:1, D0:2, D0:4, D1:1, D1:2, D1:3, D1:4, D2:0, D2:1, D2:2, D2:3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

Commit message: pcb polished
Parts:
- renumbered DISPLAY to DISPLAY1, MCU to MCU1
Connections:
- net COL0: now also MCU1.27 (GPIO21); no longer MCU1.15 (GPIO11)
- net COL1: now also MCU1.29 (GPIO22); no longer MCU1.16 (GPIO12)
- net COL2: now also MCU1.31 (GPIO26_ADC0); no longer MCU1.17 (GPIO13)
- net COL3: now also MCU1.32 (GPIO27_ADC1); no longer MCU1.19 (GPIO14)
- net COL4: now also MCU1.34 (GPIO28_ADC2); no longer MCU1.20 (GPIO15)
- net EN1_A: now also MCU1.7 (GPIO5); no longer MCU1.5 (GPIO3)
- net EN1_B: now also MCU1.6 (GPIO4); no longer MCU1.4 (GPIO2)
- net EN1_SW: now also MCU1.2 (GPIO1); no longer MCU1.31 (GPIO26_ADC0)
- net EN2_A: now also MCU1.5 (GPIO3); no longer MCU1.7 (GPIO5)
- net EN2_B: now also MCU1.4 (GPIO2); no longer MCU1.6 (GPIO4)
- net EN2_SW: now also MCU1.20 (GPIO15); no longer MCU1.32 (GPIO27_ADC1)
- net ROW0: now also MCU1.21 (GPIO16); no longer MCU1.26 (GPIO20)
- net ROW1: now also MCU1.22 (GPIO17); no longer MCU1.25 (GPIO19)
- net ROW3: now also MCU1.25 (GPIO19); no longer MCU1.22 (GPIO17)
- net ROW4: now also MCU1.26 (GPIO20); no longer MCU1.21 (GPIO16)
- net SW_WHEEL: now also MCU1.1 (GPIO0); no longer MCU1.27 (GPIO21)
Changed lines of the file:
@@
 	1    0    0    -1
 $EndComp
-Text Label 4550 4800 0    60   ~ 0
+Text Label 4550 4300 0    60   ~ 0
 ROW4
-Text Label 4550 4700 0    60   ~ 0
+Text Label 4550 4400 0    60   ~ 0
 ROW3
 Text Label 4550 4500 0    60   ~ 0
 ROW2
-Text Label 4550 4400 0    60   ~ 0
+Text Label 4550 4700 0    60   ~ 0
 ROW1
-Text Label 4550 4300 0    60   ~ 0
+Text Label 4550 4800 0    60   ~ 0
 ROW0
-Text Label 3150 3200 2    60   ~ 0
+Text Label 3150 3400 2    60   ~ 0
 EN1_B
-Text Label 3150 4300 2    60   ~ 0
+Text Label 4550 4200 0    60   ~ 0
 COL0
-Text Label 3150 4400 2    60   ~ 0
+Text Label 4550 4000 0    60   ~ 0
 COL1
-Text Label 3150 4500 2    60   ~ 0
+Text Label 4550 3800 0    60   ~ 0
 COL2
-Text Label 3150 4700 2    60   ~ 0
+Text Label 4550 3700 0    60   ~ 0
 COL3
-Text Label 3150 4800 2    60   ~ 0
+Text Label 4550 3500 0    60   ~ 0
 COL4
 Text Label 3150 3900 2    60   ~ 0
@@
 	1    0    0    -1
 $EndComp
-Text Label 3150 3500 2    60   ~ 0
+Text Label 3150 3300 2    60   ~ 0
 EN2_A
-Text Label 3150 3400 2    60   ~ 0
+Text Label 3150 3200 2    60   ~ 0
 EN2_B
-Text Label 4550 4200 0    60   ~ 0
+Text Label 3150 2900 2    60   ~ 0
 SW_WHEEL
-Text Label 4550 3800 0    60   ~ 0
-EN1_SW
 Text Label 1750 6700 3    60   ~ 0
 SCL
@@
 $EndComp
 $Comp
-L MCU_RaspberryPi_and_Boards:Pico MCU
+L MCU_RaspberryPi_and_Boards:Pico MCU1
 U 1 1 61665D33
 P 3850 3850
-F 0 "MCU" H 3850 5155 50  0000 C CNN
+F 0 "MCU1" H 3850 5155 50  0000 C CNN
 F 1 "Pico" H 3850 5064 50  0000 C CNN
 F 2 "MCU_RaspberryPi_and_Boards:RPi_Pico_SMD_TH" H 3850 4973 50  0000 C CNN
@@
 Text Label 3150 4000 2    60   ~ 0
 SCL
-Text Label 3150 3300 2    60   ~ 0
+Text Label 3150 3500 2    60   ~ 0
 EN1_A
 Text Label 1850 6700 3    60   ~ 0
@@
 	0    1    1    0
 $EndComp
-Text Label 4550 3700 0    60   ~ 0
+Text Label 3150 4800 2    60   ~ 0
 EN2_SW
 $Comp
-L userLibrary:sh1106 DISPLAY
+L userLibrary:sh1106 DISPLAY1
 U 1 1 61691921
 P 1650 6350
-F 0 "DISPLAY" H 1928 6363 50  0000 L CNN
+F 0 "DISPLAY1" H 1928 6363 50  0000 L CNN
 F 1 "sh1106" H 1928 6272 50  0000 L CNN
 F 2 "user_footprints:4pin oled display 1,3" H 1650 6350 50  0001 C CNN
@@
 	1    0    0    -1
 $EndComp
+Text Label 3150 3000 2    60   ~ 0
+EN1_SW
 $EndSCHEMATC
