File: hardware/KiCAD-Keyboard-Tutorial-master/blastpad.kicad_pcb (KiCad board)
At the start: 2 copper layers, 191.6 x 108.5 mm, 55 parts, among them SW0:0 CTRL, SW0:1 SUPER, SW0:2 ALT, SW0:4 SPACE, SW1:1 SHIFT, SW1:2 Z, SW1:3 X, SW1:4 C, SW2:0 CAPS, SW2:1 A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

Commit message: backup update
Parts:
- removed hole1 (x4): MountingHole_3.2mm_M3, MountingHole:MountingHole_3.2mm_M3
- added G***: LOGO, Blast_Logo:logo, F.Cu at (491.1, 46.8)
- added M3: MountingHole_3.2mm_M3, MountingHole:MountingHole_3.2mm_M3, F.Cu at (512.1, 127.0)
- added M3: MountingHole_3.2mm_M3, MountingHole:MountingHole_3.2mm_M3, F.Cu at (363.5, 127.0)
- added M3: MountingHole_3.2mm_M3, MountingHole:MountingHole_3.2mm_M3, F.Cu at (472.0, 78.1)
- added M3: MountingHole_3.2mm_M3, MountingHole:MountingHole_3.2mm_M3, F.Cu at (512.0, 28.5)
- added M3: MountingHole_3.2mm_M3, MountingHole:MountingHole_3.2mm_M3, F.Cu at (330.4, 28.5)
- added M3: MountingHole_3.2mm_M3, MountingHole:MountingHole_3.2mm_M3, F.Cu at (330.4, 95.3)
- D0:0, D0:1, D0:2, D0:4, D1:1, D1:2, D1:3, D1:4, D2:0, D2:1, D2:2, D2:3, D2:4, D3:0, D3:1, D3:2, D3:3, D3:4, D4:0, D4:1, D4:2, D4:3, D4:4: footprint footprints:DIODE -> user_footprints:DIODE
Routing:
- net /EN1_A: track 229.1 -> 221.2 mm
Other:
- board size 191.6 x 108.5 mm -> 191.7 x 108.5 mm
- board text added: "BlastPad/Rafał Buchner/2021"
