File: hardware/KiCAD-Keyboard-Tutorial-master/blastpad.sch (KiCad schematic (older format))
At the start: 51 parts, among them SW0:0 CTRL, SW0:1 SUPER, SW0:2 ALT, SW0:4 SPACE, SW1:1 SHIFT, SW1:2 Z, SW1:3 X, SW1:4 C, SW2:0 CAPS, SW2:1 A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

Commit message: backup update
Parts:
- D0:0, D0:1, D0:2, D0:4, D1:1, D1:2, D1:3, D1:4, D2:0, D2:1, D2:2, D2:3, D2:4, D3:0, D3:1, D3:2, D3:3, D3:4, D4:0, D4:1, D4:2, D4:3, D4:4: footprint footprints:DIODE -> user_footprints:DIODE
Changed lines of the file:
@@
 F 0 "D0:2" H 8700 5050 40  0000 C CNN
 F 1 "D" H 8700 4850 40  0000 C CNN
-F 2 "footprints:DIODE" H 8700 4950 60  0001 C CNN
+F 2 "user_footprints:DIODE" H 8700 4950 60  0001 C CNN
 F 3 "" H 8700 4950 60  0001 C CNN
 	1    8700 4950
@@
 F 0 "D0:1" H 7900 5050 40  0000 C CNN
 F 1 "D" H 7900 4850 40  0000 C CNN
-F 2 "footprints:DIODE" H 7900 4950 60  0001 C CNN
+F 2 "user_footprints:DIODE" H 7900 4950 60  0001 C CNN
 F 3 "" H 7900 4950 60  0001 C CNN
 	1    7900 4950
@@
 F 0 "D0:0" H 7100 5050 40  0000 C CNN
 F 1 "D" H 7100 4850 40  0000 C CNN
-F 2 "footprints:DIODE" H 7100 4950 60  0001 C CNN
+F 2 "user_footprints:DIODE" H 7100 4950 60  0001 C CNN
 F 3 "" H 7100 4950 60  0001 C CNN
 	1    7100 4950
@@
 F 0 "D1:4" H 10300 4200 40  0000 C CNN
 F 1 "D" H 10300 4000 40  0000 C CNN
-F 2 "footprints:DIODE" H 10300 4100 60  0001 C CNN
+F 2 "user_footprints:DIODE" H 10300 4100 60  0001 C CNN
 F 3 "" H 10300 4100 60  0001 C CNN
 	1    10300 4100
@@
 F 0 "D3:4" H 10300 2500 40  0000 C CNN
 F 1 "D" H 10300 2300 40  0000 C CNN
-F 2 "footprints:DIODE" H 10300 2400 60  0001 C CNN
+F 2 "user_footprints:DIODE" H 10300 2400 60  0001 C CNN
 F 3 "" H 10300 2400 60  0001 C CNN
 	1    10300 2400
@@
 F 0 "D2:4" H 10300 3350 40  0000 C CNN
 F 1 "D" H 10300 3150 40  0000 C CNN
-F 2 "footprints:DIODE" H 10300 3250 60  0001 C CNN
+F 2 "user_footprints:DIODE" H 10300 3250 60  0001 C CNN
 F 3 "" H 10300 3250 60  0001 C CNN
 	1    10300 3250
@@
 F 0 "D4:2" H 8700 1650 40  0000 C CNN
 F 1 "D" H 8700 1450 40  0000 C CNN
-F 2 "footprints:DIODE" H 8700 1550 60  0001 C CNN
+F 2 "user_footprints:DIODE" H 8700 1550 60  0001 C CNN
 F 3 "" H 8700 1550 60  0001 C CNN
 	1    8700 1550
@@
 F 0 "D4:3" H 9500 1650 40  0000 C CNN
 F 1 "D" H 9500 1450 40  0000 C CNN
-F 2 "footprints:DIODE" H 9500 1550 60  0001 C CNN
+F 2 "user_footprints:DIODE" H 9500 1550 60  0001 C CNN
 F 3 "" H 9500 1550 60  0001 C CNN
 	1    9500 1550
@@
 F 0 "D0:4" H 10300 5050 40  0000 C CNN
 F 1 "D" H 10300 4850 40  0000 C CNN
-F 2 "footprints:DIODE" H 10300 4950 60  0001 C CNN
+F 2 "user_footprints:DIODE" H 10300 4950 60  0001 C CNN
 F 3 "" H 10300 4950 60  0001 C CNN
 	1    10300 4950
@@
 F 0 "D4:4" H 10300 1650 40  0000 C CNN
 F 1 "D" H 10300 1450 40  0000 C CNN
-F 2 "footprints:DIODE" H 10300 1550 60  0001 C CNN
+F 2 "user_footprints:DIODE" H 10300 1550 60  0001 C CNN
 F 3 "" H 10300 1550 60  0001 C CNN
 	1    10300 1550
@@
 F 0 "D1:1" H 7900 4200 40  0000 C CNN
 F 1 "D" H 7900 4000 40  0000 C CNN
-F 2 "footprints:DIODE" H 7900 4100 60  0001 C CNN
+F 2 "user_footprints:DIODE" H 7900 4100 60  0001 C CNN
 F 3 "" H 7900 4100 60  0001 C CNN
 	1    7900 4100
@@
 F 0 "D3:0" H 7100 2500 40  0000 C CNN
 F 1 "D" H 7100 2300 40  0000 C CNN
-F 2 "footprints:DIODE" H 7100 2400 60  0001 C CNN
+F 2 "user_footprints:DIODE" H 7100 2400 60  0001 C CNN
 F 3 "" H 7100 2400 60  0001 C CNN
 	1    7100 2400
@@
 F 0 "D2:0" H 7100 3350 40  0000 C CNN
 F 1 "D" H 7100 3150 40  0000 C CNN
-F 2 "footprints:DIODE" H 7100 3250 60  0001 C CNN
+F 2 "user_footprints:DIODE" H 7100 3250 60  0001 C CNN
 F 3 "" H 7100 3250 60  0001 C CNN
 	1    7100 3250
@@
 F 0 "D2:1" H 7900 3350 40  0000 C CNN
 F 1 "D" H 7900 3150 40  0000 C CNN
-F 2 "footprints:DIODE" H 7900 3250 60  0001 C CNN
+F 2 "user_footprints:DIODE" H 7900 3250 60  0001 C CNN
 F 3 "" H 7900 3250 60  0001 C CNN
 	1    7900 3250
@@
 F 0 "D3:1" H 7900 2500 40  0000 C CNN
 F 1 "D" H 7900 2300 40  0000 C CNN
-F 2 "footprints:DIODE" H 7900 2400 60  0001 C CNN
+F 2 "user_footprints:DIODE" H 7900 2400 60  0001 C CNN
 F 3 "" H 7900 2400 60  0001 C CNN
 	1    7900 2400
@@
 F 0 "D1:3" H 9500 4200 40  0000 C CNN
 F 1 "D" H 9500 4000 40  0000 C CNN
-F 2 "footprints:DIODE" H 9500 4100 60  0001 C CNN
+F 2 "user_footprints:DIODE" H 9500 4100 60  0001 C CNN
 F 3 "" H 9500 4100 60  0001 C CNN
 	1    9500 4100
@@
 F 0 "D3:3" H 9500 2500 40  0000 C CNN
 F 1 "D" H 9500 2300 40  0000 C CNN
-F 2 "footprints:DIODE" H 9500 2400 60  0001 C CNN
+F 2 "user_footprints:DIODE" H 9500 2400 60  0001 C CNN
 F 3 "" H 9500 2400 60  0001 C CNN
 	1    9500 2400
@@
 F 0 "D2:3" H 9500 3350 40  0000 C CNN
 F 1 "D" H 9500 3150 40  0000 C CNN
-F 2 "footprints:DIODE" H 9500 3250 60  0001 C CNN
+F 2 "user_footprints:DIODE" H 9500 3250 60  0001 C CNN
 F 3 "" H 9500 3250 60  0001 C CNN
 	1    9500 3250
@@
 F 0 "D4:1" H 7900 1650 40  0000 C CNN
 F 1 "D" H 7900 1450 40  0000 C CNN
-F 2 "footprints:DIODE" H 7900 1550 60  0001 C CNN
+F 2 "user_footprints:DIODE" H 7900 1550 60  0001 C CNN
 F 3 "" H 7900 1550 60  0001 C CNN
 	1    7900 1550
@@
 F 0 "D4:0" H 7100 1650 40  0000 C CNN
 F 1 "D" H 7100 1450 40  0000 C CNN
-F 2 "footprints:DIODE" H 7100 1550 60  0001 C CNN
+F 2 "user_footprints:DIODE" H 7100 1550 60  0001 C CNN
 F 3 "" H 7100 1550 60  0001 C CNN
 	1    7100 1550
@@
 F 0 "D2:2" H 8700 3350 40  0000 C CNN
 F 1 "D" H 8700 3150 40  0000 C CNN
-F 2 "footprints:DIODE" H 8700 3250 60  0001 C CNN
+F 2 "user_footprints:DIODE" H 8700 3250 60  0001 C CNN
 F 3 "" H 8700 3250 60  0001 C CNN
 	1    8700 3250
@@
 F 0 "D3:2" H 8700 2500 40  0000 C CNN
 F 1 "D" H 8700 2300 40  0000 C CNN
-F 2 "footprints:DIODE" H 8700 2400 60  0001 C CNN
+F 2 "user_footprints:DIODE" H 8700 2400 60  0001 C CNN
 F 3 "" H 8700 2400 60  0001 C CNN
 	1    8700 2400
@@
 F 0 "D1:2" H 8700 4200 40  0000 C CNN
 F 1 "D" H 8700 4000 40  0000 C CNN
-F 2 "footprints:DIODE" H 8700 4100 60  0001 C CNN
+F 2 "user_footprints:DIODE" H 8700 4100 60  0001 C CNN
 F 3 "" H 8700 4100 60  0001 C CNN
 	1    8700 4100
